File: plate/discipline-plate.kicad_pcb (KiCad board)
At the start: 2 copper layers, 304.9 x 95.3 mm, 2 parts

Commit message: Add ISO support; add 2x1.25u + 0.5u blocker layout right of spacebar
Other:
- outline, holes or cut-outs redrawn
- board text added: "coseyfannitutti 2019 V1.5 by piit79 2021"
- board text removed: "coseyfannitutti 2019 rev1"
