File: discipline-pcb.kicad_pcb (KiCad board)
At the start: 2 copper layers, 304.9 x 122.8 mm, 180 parts, among them J1 AVR-ISP-6, SW1 KEYSW, SW10 KEYSW, SW11 KEYSW, SW12 KEYSW, SW13 KEYSW, SW14 KEYSW, SW15 KEYSW, SW16 KEYSW, SW17 KEYSW, SW18 KEYSW, SW19 KEYSW, SW2 KEYSW, SW20 KEYSW, SW21 KEYSW, SW22 KEYSW, SW23 KEYSW, SW24 KEYSW, SW25 KEYSW, SW26 KEYSW, SW27 KEYSW, SW28 KEYSW, SW29 KEYSW, SW3 KEYSW, SW30 KEYSW, SW31 KEYSW, SW32 KEYSW, SW33 KEYSW, SW34 KEYSW, SW35 KEYSW, SW36 KEYSW, SW37 KEYSW, SW38 KEYSW, SW39 KEYSW, SW4 KEYSW, SW40 KEYSW, SW41 KEYSW, SW42 KEYSW, SW43 KEYSW, SW44 KEYSW, SW45 KEYSW, SW46 KEYSW, SW47 KEYSW, SW48 KEYSW, SW49 KEYSW, SW5 KEYSW, SW50 KEYSW, SW51 KEYSW, SW52 KEYSW, SW53 KEYSW, SW54 KEYSW, SW55 KEYSW, SW56 KEYSW, SW57 KEYSW, SW58 KEYSW, SW59 KEYSW, SW6 KEYSW, SW60 KEYSW, SW61 KEYSW, SW62 KEYSW, SW63 KEYSW, SW64 KEYSW, SW65 KEYSW, SW66 KEYSW, SW67 KEYSW, SW68 KEYSW, SW69 KEYSW, SW7 KEYSW, SW70 KEYSW, SW71 KEYSW, SW72 KEYSW, SW73 KEYSW, SW74 KEYSW, SW8 KEYSW, SW9 KEYSW, U1 ATmega32A-PU, Y1 Crystal

Commit message: Add ISO support; add 2x1.25u + 0.5u blocker layout right of spacebar
Parts:
- added D78: , cftkb:D_DO-35_SOD27_P5.08mm_Horizontal, F.Cu at (96.7, 147.9)
- added REF**: MountingHole_2.2mm_M2_Pad, MountingHole:MountingHole_2.2mm_M2_Pad, F.Cu at (206.2, 80.5)
- added REF**: MountingHole_2.2mm_M2_Pad, MountingHole:MountingHole_2.2mm_M2_Pad, F.Cu at (206.2, 61.7)
- added SW75: KEYSW, cftkb:SW_Cherry_MX1A_ISOEnter_PCB_ReversedStabilizer, F.Cu at (330.2, 118.3)
- added SW76: KEYSW, cftkb:SW_Cherry_MX1A_1.00u_PCB-NOSCREEN, F.Cu at (308.8, 127.8)
- added SW77: KEYSW, cftkb:SW_Cherry_MX1A_1.25u_PCBNOSCREEN, F.Cu at (68.3, 146.8)
- added SW78: KEYSW, cftkb:SW_Cherry_MX1A_1.00u_PCB-NOSCREEN, F.Cu at (89.7, 146.8)
- added SW79: KEYSW, cftkb:SW_Cherry_MX1A_1.25u_PCBNOSCREEN, F.Cu at (258.8, 165.9)
- added SW80: KEYSW, cftkb:SW_Cherry_MX1A_1.25u_PCBNOSCREEN, F.Cu at (282.6, 165.9)
- REF**: value 6.25U -> 6.25u
- ST72: value 7U -> 7u
- moved G*** 2.40 mm to (153.1, 164.9) (x2)
- moved REF** 0.73 mm to (354.7, 80.5)
- moved REF** 0.73 mm to (57.8, 80.5)
- moved REF** 0.72 mm to (354.7, 61.7)
- moved REF** 0.72 mm to (57.8, 61.7)
Routing:
- net row3: track 287.2 -> 392.6 mm
- net Net-(D78-Pad2): track 0.00 -> 16.5 mm
- net col13: track 146.9 -> 163.3 mm
- net Net-(D43-Pad2): track 140.6 -> 155.0 mm
- net Net-(D29-Pad2): track 117.7 -> 128.1 mm
- net GND: track 241.1 -> 231.5 mm, vias 36 -> 39
- net Net-(D45-Pad2): track 76.5 -> 85.7 mm
- net col12: track 182.7 -> 189.6 mm
- net col0: track 355.0 -> 361.8 mm
- net Net-(D60-Pad2): track 102.3 -> 105.2 mm
- net col1: track 317.2 -> 315.0 mm
- net Net-(D64-Pad2): track 187.5 -> 189.5 mm
- net col5: track 271.6 -> 270.0 mm
- net Net-(D56-Pad2): track 145.3 -> 146.8 mm
- net col6: track 279.4 -> 278.3 mm
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Other:
- net class Power added: clearance 0.2, trace_width 0.4, via_dia 0.8, via_drill 0.4
- board text added: "1.25u"
- board text added: "1.25u ISO"
- board text added: "1.5u"
- board text added: "1u"
- board text added: "1u ISO"
- board text added: "2.25u ANSI"
- board text added: "ANSI ENTER"
- board text added: "ISO"
- board text added: "ISO ENTER"
- board text added: "coseyfannitutti 2019 V1.5 by piit79 2021"
- board text removed: "1.25U"
- board text removed: "1.5U"
- board text removed: "1U"
- board text removed: "coseyfannitutti 2019 rev1"

Commit message: Add support for a rotary encoder in top right position
Parts:
- added SW81: Rotary_Encoder_Switch, cftkb:RotaryEncoder_Alps_EC11E-Switch_Vertical_H20mm-for-MX, F.Cu at (346.6, 102.3)
- SW63, SW64: footprint cftkb:SW_Cherry_MX1A_1.00u_PCB-NOSCREEN -> cftkb:SW_Cherry_MX1A_1.25u_PCBNOSCREEN
- moved R7 7.62 mm to (288.8, 63.1), turned to 0 degrees
Connections:
- U1 pad 14: Net-(U1-Pad14) -> EN1
- U1 pad 15: Net-(U1-Pad15) -> EN2
- U1 pad 29: Net-(U1-Pad29) -> (no net)
- U1 pad 32: Net-(U1-Pad32) -> (no net)
- U1 pad 33: Net-(U1-Pad33) -> (no net)
- U1 pad 34: Net-(U1-Pad34) -> (no net)
- U1 pad 35: Net-(U1-Pad35) -> (no net)
- USB1 pad A8: Net-(USB1-PadA8) -> (no net)
- USB1 pad B8: Net-(USB1-PadB8) -> (no net)
Routing:
- net EN2: track 0.00 -> 47.9 mm, vias 0 -> 1
- net EN1: track 0.00 -> 47.6 mm, vias 0 -> 1
- net +5V: track 147.9 -> 114.3 mm
- net reset: track 128.8 -> 119.0 mm, vias 2 -> 1
- net Net-(D15-Pad2): track 78.0 -> 83.0 mm
- net col11: track 213.9 -> 210.6 mm
- net col9: track 260.1 -> 256.9 mm
- net col14: track 107.8 -> 110.8 mm
- net col13: track 163.3 -> 160.9 mm
- net col12: track 189.6 -> 187.2 mm
- net col10: track 251.0 -> 248.6 mm
- net col8: track 246.3 -> 244.0 mm
- net col6: track 278.3 -> 276.0 mm
- net col5: track 270.0 -> 267.7 mm
- net col7: track 269.0 -> 266.7 mm
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Other:
- board text added: "coseyfannitutti 2019 V1.5b by piit79 2021"
- board text removed: "coseyfannitutti 2019 V1.5 by piit79 2021"
