File: discipline-pcb.sch (KiCad schematic (older format))
At the start: 164 parts, among them J1 AVR-ISP-6, SW1 KEYSW, SW10 KEYSW, SW11 KEYSW, SW12 KEYSW, SW13 KEYSW, SW14 KEYSW, SW15 KEYSW, SW16 KEYSW, SW17 KEYSW, SW18 KEYSW, SW19 KEYSW, SW2 KEYSW, SW20 KEYSW, SW21 KEYSW, SW22 KEYSW, SW23 KEYSW, SW24 KEYSW, SW25 KEYSW, SW26 KEYSW, SW27 KEYSW, SW28 KEYSW, SW29 KEYSW, SW3 KEYSW, SW30 KEYSW, SW31 KEYSW, SW32 KEYSW, SW33 KEYSW, SW34 KEYSW, SW35 KEYSW, SW36 KEYSW, SW37 KEYSW, SW38 KEYSW, SW39 KEYSW, SW4 KEYSW, SW40 KEYSW, SW41 KEYSW, SW42 KEYSW, SW43 KEYSW, SW44 KEYSW, SW45 KEYSW, SW46 KEYSW, SW47 KEYSW, SW48 KEYSW, SW49 KEYSW, SW5 KEYSW, SW50 KEYSW, SW51 KEYSW, SW52 KEYSW, SW53 KEYSW, SW54 KEYSW, SW55 KEYSW, SW56 KEYSW, SW57 KEYSW, SW58 KEYSW, SW59 KEYSW, SW6 KEYSW, SW60 KEYSW, SW61 KEYSW, SW62 KEYSW, SW63 KEYSW, SW64 KEYSW, SW65 KEYSW, SW66 KEYSW, SW67 KEYSW, SW68 KEYSW, SW69 KEYSW, SW7 KEYSW, SW70 KEYSW, SW71 KEYSW, SW72 KEYSW, SW73 KEYSW, SW74 KEYSW, SW8 KEYSW, SW9 KEYSW, U1 ATmega32A-PU, Y1 Crystal

Commit message: Add ISO support; add 2x1.25u + 0.5u blocker layout right of spacebar
Parts:
- added D78: (no value), cftkb:D_DO-35_SOD27_P5.08mm_Horizontal, symbol Device:D
- added SW75: KEYSW, cftkb:SW_Cherry_MX1A_ISOEnter_PCB_ReversedStabilizer, symbol discipline-pcb-rescue:KEYSW-keyboard_parts
- added SW76, SW78: KEYSW, cftkb:SW_Cherry_MX1A_1.00u_PCB-NOSCREEN, symbol discipline-pcb-rescue:KEYSW-keyboard_parts
- added SW77, SW79, SW80: KEYSW, cftkb:SW_Cherry_MX1A_1.25u_PCBNOSCREEN, symbol discipline-pcb-rescue:KEYSW-keyboard_parts
- BOOT1, RESET1: symbol keyboard_parts:SW_PUSH -> discipline-pcb-rescue:SW_PUSH-keyboard_parts
- J1: symbol Connector:AVR-ISP-6 -> discipline-pcb-rescue:AVR-ISP-6-Connector
- SW1, SW10, SW11, SW12, SW13, SW14, SW15, SW16, SW17, SW18, SW19, SW2, SW20, SW21, SW22, SW23, SW24, SW25, SW26, SW27, SW28, SW29, SW3, SW30, SW31, SW32, SW33, SW34, SW35, SW36, SW37, SW38, SW39, SW4, SW40, SW41, SW42, SW43, SW44, SW45, SW46, SW47, SW48, SW49, SW5, SW50, SW51, SW52, SW53, SW54, SW55, SW56, SW57, SW58, SW59, SW6, SW60, SW61, SW62, SW63, SW64, SW65, SW66, SW67, SW68, SW69, SW7, SW70, SW71, SW72, SW73, SW74, SW8, SW9: symbol keyboard_parts:KEYSW -> discipline-pcb-rescue:KEYSW-keyboard_parts
- U1: symbol MCU_Microchip_ATmega:ATmega32A-PU -> discipline-pcb-rescue:ATmega32A-PU-MCU_Microchip_ATmega
- USB1: symbol Type-C:USB_C_GCT_USB4085 -> discipline-pcb-rescue:USB_C_GCT_USB4085-Type-C
Connections:
- wire segments 342 -> 360

Commit message: Add support for a rotary encoder in top right position
Parts:
- added SW81: Rotary_Encoder_Switch, cftkb:RotaryEncoder_Alps_EC11E-Switch_Vertical_H20mm-for-MX, symbol Device:Rotary_Encoder_Switch
- BOOT1, RESET1: symbol discipline-pcb-rescue:SW_PUSH-keyboard_parts -> discipline-pcb-rescue:SW_PUSH-keyboard_parts-discipline-pcb-rescue
- C1, C2: footprint cftkb:D_DO-35_SOD27_P5.08mm_Horizontal -> cftkb:C_Disc_D3.0mm_W1.6mm_P2.50mm
- C3: footprint cftkb:D_DO-35_SOD27_P5.08mm_Horizontal -> cftkb:CP_Radial_D4.0mm_P1.50mm
- C4, C5: footprint cftkb:D_DO-35_SOD27_P5.08mm_Horizontal -> cftkb:C_Disc_D4.3mm_W1.9mm_P5.00mm
- J1: symbol discipline-pcb-rescue:AVR-ISP-6-Connector -> discipline-pcb-rescue:AVR-ISP-6-Connector-discipline-pcb-rescue
- SW1, SW10, SW11, SW12, SW13, SW14, SW15, SW16, SW17, SW18, SW19, SW2, SW20, SW21, SW22, SW23, SW24, SW25, SW26, SW27, SW28, SW29, SW3, SW30, SW31, SW32, SW33, SW34, SW35, SW36, SW37, SW38, SW39, SW4, SW40, SW41, SW42, SW43, SW44, SW45, SW46, SW47, SW48, SW49, SW5, SW50, SW51, SW52, SW53, SW54, SW55, SW56, SW57, SW58, SW59, SW6, SW60, SW61, SW62, SW63, SW64, SW65, SW66, SW67, SW68, SW69, SW7, SW70, SW71, SW72, SW73, SW74, SW75, SW76, SW77, SW78, SW79, SW8, SW80, SW9: symbol discipline-pcb-rescue:KEYSW-keyboard_parts -> discipline-pcb-rescue:KEYSW-keyboard_parts-discipline-pcb-rescue
- U1: symbol discipline-pcb-rescue:ATmega32A-PU-MCU_Microchip_ATmega -> discipline-pcb-rescue:ATmega32A-PU-MCU_Microchip_ATmega-discipline-pcb-rescue
- USB1: symbol discipline-pcb-rescue:USB_C_GCT_USB4085-Type-C -> discipline-pcb-rescue:USB_C_GCT_USB4085-Type-C-discipline-pcb-rescue
Connections:
- net GND: now also SW81.C
- net col14: now also SW81.S1
- net at D15.2 (A), SW15.2: now also SW81.S2
- net EN1: now reaches U1.14 (PD0)
- net EN1: now also SW81.B
- net EN2: now reaches U1.15 (PD1)
- net EN2: now also SW81.A
- no-connect marks 9 -> 7
Other:
- moved on the sheet: R7
