File: bottom/discipline-bottom.kicad_pcb (KiCad board)
At the start: 2 copper layers, 304.9 x 122.8 mm, 20 parts

Commit message: Update bottom large logo for both copper and mask
Parts:
- removed the G*** at (209.4, 112.7)
- added G***: LOGO, cftkb:DISCIPLINE_LARGE_COPPER_MASK, B.Cu at (209.4, 112.7)
